File: wifilight-leds-cheaper.sch (EAGLE design)
At the start: 48 parts, among them Q1 BUK98180-100A, Q2 BUK98180-100A, Q3 BUK98180-100A, Q4 BUK98180-100A, U2 PCA9685

Commit message: add SCL & SDA pins pogopins for programming
Parts:
- added TPRX, TPTX: TEST-POINT3X5, SparkFun-Passives:TEST-POINT3X5
Connections:
- removed net N$29: MPU.REST
- removed net N$32: MPU.GPIO4
- new net RXD: MPU.RXD, TPRX.1
- new net TXD: MPU.TXD, TPTX.1
- net RESET: now also MPU.REST; no longer MPU.TXD
- net THINKING: now also MPU.GPIO4; no longer MPU.RXD
Changed lines of the file:
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@@
 <part name="H1" library="LilyPad-Wearables" deviceset="SEW_HOLE" device=""/>
 <part name="TPGND" library="SparkFun-Passives" deviceset="TEST-POINT" device="3X5"/>
+<part name="TPTX" library="SparkFun-Passives" deviceset="TEST-POINT" device="3X5"/>
+<part name="TPRX" library="SparkFun-Passives" deviceset="TEST-POINT" device="3X5"/>
 </parts>
 <sheets>
@@
 <instance part="H1" gate="G$1" x="-149.86" y="45.72" rot="R180"/>
 <instance part="TPGND" gate="G$1" x="-119.38" y="45.72"/>
+<instance part="TPTX" gate="G$1" x="-78.74" y="-43.18"/>
+<instance part="TPRX" gate="G$1" x="-78.74" y="-53.34"/>
 </instances>
 <busses>
@@
 </segment>
 <segment>
-<pinref part="MPU" gate="G$1" pin="RXD"/>
-<wire x1="129.54" y1="66.04" x2="116.84" y2="66.04" width="0.1524" layer="91"/>
-<label x="119.38" y="66.04" size="1.778" layer="95"/>
+<pinref part="MPU" gate="G$1" pin="GPIO4"/>
+<wire x1="116.84" y1="63.5" x2="129.54" y2="63.5" width="0.1524" layer="91"/>
+<label x="119.38" y="63.5" size="1.778" layer="95"/>
 </segment>
 </net>
@@
 </segment>
 </net>
-<net name="N$29" class="0">
+<net name="RESET" class="0">
 <segment>
 <pinref part="MPU" gate="G$1" pin="REST"/>
@@
 </segment>
 </net>
-<net name="RESET" class="0">
+<net name="N$33" class="0">
+<segment>
+<pinref part="MPU" gate="G$1" pin="GPIO0"/>
+<wire x1="129.54" y1="58.42" x2="116.84" y2="58.42" width="0.1524" layer="91"/>
+<label x="119.38" y="58.42" size="1.778" layer="95"/>
+</segment>
+</net>
+<net name="N$34" class="0">
+<segment>
+<pinref part="MPU" gate="G$1" pin="GPIO2"/>
+<wire x1="116.84" y1="55.88" x2="129.54" y2="55.88" width="0.1524" layer="91"/>
+<label x="119.38" y="55.88" size="1.778" layer="95"/>
+</segment>
+</net>
+<net name="N$35" class="0">
+<segment>
+<pinref part="MPU" gate="G$1" pin="GPIO15"/>
+<wire x1="129.54" y1="53.34" x2="116.84" y2="53.34" width="0.1524" layer="91"/>
+<label x="119.38" y="53.34" size="1.778" layer="95"/>
+</segment>
+</net>
+<net name="N$36" class="0">
+<segment>
+<pinref part="MPU" gate="G$1" pin="GPIO5"/>
+<wire x1="116.84" y1="60.96" x2="129.54" y2="60.96" width="0.1524" layer="91"/>
+<label x="119.38" y="60.96" size="1.778" layer="95"/>
+</segment>
+</net>
+<net name="TXD" class="0">
 <segment>
 <pinref part="MPU" gate="G$1" pin="TXD"/>
@@
 <label x="119.38" y="68.58" size="1.778" layer="95"/>
 </segment>
-</net>
-<net name="N$32" class="0">
-<segment>
-<pinref part="MPU" gate="G$1" pin="GPIO4"/>
-<wire x1="116.84" y1="63.5" x2="129.54" y2="63.5" width="0.1524" layer="91"/>
-<label x="119.38" y="63.5" size="1.778" layer="95"/>
-</segment>
-</net>
-<net name="N$33" class="0">
-<segment>
-<pinref part="MPU" gate="G$1" pin="GPIO0"/>
-<wire x1="129.54" y1="58.42" x2="116.84" y2="58.42" width="0.1524" layer="91"/>
-<label x="119.38" y="58.42" size="1.778" layer="95"/>
-</segment>
-</net>
-<net name="N$34" class="0">
-<segment>
-<pinref part="MPU" gate="G$1" pin="GPIO2"/>
-<wire x1="116.84" y1="55.88" x2="129.54" y2="55.88" width="0.1524" layer="91"/>
-<label x="119.38" y="55.88" size="1.778" layer="95"/>
-</segment>
-</net>
-<net name="N$35" class="0">
-<segment>
-<pinref part="MPU" gate="G$1" pin="GPIO15"/>
-<wire x1="129.54" y1="53.34" x2="116.84" y2="53.34" width="0.1524" layer="91"/>
-<label x="119.38" y="53.34" size="1.778" layer="95"/>
-</segment>
-</net>
-<net name="N$36" class="0">
-<segment>
-<pinref part="MPU" gate="G$1" pin="GPIO5"/>
-<wire x1="116.84" y1="60.96" x2="129.54" y2="60.96" width="0.1524" layer="91"/>
-<label x="119.38" y="60.96" size="1.778" layer="95"/>
-</segment>
-</net>
+<segment>
+<wire x1="-104.14" y1="-43.18" x2="-78.74" y2="-43.18" width="0.1524" layer="91"/>
+<label x="-99.06" y="-43.18" size="1.778" layer="95"/>
+<pinref part="TPTX" gate="G$1" pin="1"/>
+</segment>
+</net>
+<net name="RXD" class="0">
+<segment>
+<pinref part="MPU" gate="G$1" pin="RXD"/>
+<wire x1="129.54" y1="66.04" x2="116.84" y2="66.04" width="0.1524" layer="91"/>
+<label x="119.38" y="66.04" size="1.778" layer="95"/>
+</segment>
+<segment>
+<wire x1="-78.74" y1="-53.34" x2="-104.14" y2="-53.34" width="0.1524" layer="91"/>
+<label x="-99.06" y="-53.34" size="1.778" layer="95"/>
+<pinref part="TPRX" gate="G$1" pin="1"/>
+</segment>
+</net>

Commit message: add TXD, RXD & GPIO0 pins pogopins for programming
Parts:
- added TPGPIO0: TEST-POINT3X5, SparkFun-Passives:TEST-POINT3X5
Connections:
- removed net N$33: MPU.GPIO0
- removed net N$35: MPU.GPIO15
- new net DISCO: MPU.GPIO4
- new net GPIO0: MPU.GPIO0, TPGPIO0.1
- net THINKING: now also MPU.GPIO15; no longer MPU.GPIO4
Changed lines of the file:
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@@
 <part name="TPTX" library="SparkFun-Passives" deviceset="TEST-POINT" device="3X5"/>
 <part name="TPRX" library="SparkFun-Passives" deviceset="TEST-POINT" device="3X5"/>
+<part name="TPGPIO0" library="SparkFun-Passives" deviceset="TEST-POINT" device="3X5"/>
 </parts>
 <sheets>
@@
 <instance part="TPTX" gate="G$1" x="-78.74" y="-43.18"/>
 <instance part="TPRX" gate="G$1" x="-78.74" y="-53.34"/>
+<instance part="TPGPIO0" gate="G$1" x="-78.74" y="-63.5"/>
 </instances>
 <busses>
@@
 </segment>
 <segment>
-<pinref part="MPU" gate="G$1" pin="GPIO4"/>
-<wire x1="116.84" y1="63.5" x2="129.54" y2="63.5" width="0.1524" layer="91"/>
-<label x="119.38" y="63.5" size="1.778" layer="95"/>
+<pinref part="MPU" gate="G$1" pin="GPIO15"/>
+<wire x1="129.54" y1="53.34" x2="116.84" y2="53.34" width="0.1524" layer="91"/>
+<label x="119.38" y="53.34" size="1.778" layer="95"/>
 </segment>
 </net>
@@
 </segment>
 </net>
-<net name="N$33" class="0">
+<net name="GPIO0" class="0">
 <segment>
 <pinref part="MPU" gate="G$1" pin="GPIO0"/>
@@
 <label x="119.38" y="58.42" size="1.778" layer="95"/>
 </segment>
+<segment>
+<wire x1="-78.74" y1="-63.5" x2="-104.14" y2="-63.5" width="0.1524" layer="91"/>
+<label x="-99.06" y="-63.5" size="1.778" layer="95"/>
+<pinref part="TPGPIO0" gate="G$1" pin="1"/>
+</segment>
 </net>
 <net name="N$34" class="0">
@@
 </segment>
 </net>
-<net name="N$35" class="0">
-<segment>
-<pinref part="MPU" gate="G$1" pin="GPIO15"/>
-<wire x1="129.54" y1="53.34" x2="116.84" y2="53.34" width="0.1524" layer="91"/>
-<label x="119.38" y="53.34" size="1.778" layer="95"/>
-</segment>
-</net>
 <net name="N$36" class="0">
 <segment>
@@
 </segment>
 </net>
+<net name="DISCO" class="0">
+<segment>
+<pinref part="MPU" gate="G$1" pin="GPIO4"/>
+<wire x1="116.84" y1="63.5" x2="129.54" y2="63.5" width="0.1524" layer="91"/>
+<label x="119.38" y="63.5" size="1.778" layer="95"/>
+</segment>
+</net>

Commit message: add GPIO2 pins pogopins for programming
Parts:
- added TPCHPD, TPGPIO2: TEST-POINT3X5, SparkFun-Passives:TEST-POINT3X5
Connections:
- removed net N$27: MPU.CH_PD
- removed net N$34: MPU.GPIO2
- new net CH_PD: MPU.CH_PD, TPCHPD.1
- new net GPIO2: MPU.GPIO2, TPGPIO2.1
Changed lines of the file:
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@@
 <part name="TPRX" library="SparkFun-Passives" deviceset="TEST-POINT" device="3X5"/>
 <part name="TPGPIO0" library="SparkFun-Passives" deviceset="TEST-POINT" device="3X5"/>
+<part name="TPCHPD" library="SparkFun-Passives" deviceset="TEST-POINT" device="3X5"/>
+<part name="TPGPIO2" library="SparkFun-Passives" deviceset="TEST-POINT" device="3X5"/>
 </parts>
 <sheets>
@@
 <instance part="TPRX" gate="G$1" x="-78.74" y="-53.34"/>
 <instance part="TPGPIO0" gate="G$1" x="-78.74" y="-63.5"/>
+<instance part="TPCHPD" gate="G$1" x="-78.74" y="-73.66"/>
+<instance part="TPGPIO2" gate="G$1" x="-78.74" y="-83.82"/>
 </instances>
 <busses>
@@
 </segment>
 </net>
-<net name="N$27" class="0">
+<net name="CH_PD" class="0">
 <segment>
 <pinref part="MPU" gate="G$1" pin="CH_PD"/>
@@
 <label x="76.2" y="63.5" size="1.778" layer="95"/>
 </segment>
+<segment>
+<wire x1="-78.74" y1="-73.66" x2="-104.14" y2="-73.66" width="0.1524" layer="91"/>
+<label x="-99.06" y="-73.66" size="1.778" layer="95"/>
+<pinref part="TPCHPD" gate="G$1" pin="1"/>
+</segment>
 </net>
 <net name="N$28" class="0">
@@
 </segment>
 </net>
-<net name="N$34" class="0">
+<net name="GPIO2" class="0">
 <segment>
 <pinref part="MPU" gate="G$1" pin="GPIO2"/>
@@
 <label x="119.38" y="55.88" size="1.778" layer="95"/>
 </segment>
-</net>
+<segment>
+<wire x1="-78.74" y1="-83.82" x2="-104.14" y2="-83.82" width="0.1524" layer="91"/>
+<label x="-99.06" y="-83.82" size="1.778" layer="95"/>
+<pinref part="TPGPIO2" gate="G$1" pin="1"/>
+</segment>
+</net>
