File: wifilight.brd (EAGLE design)
At the start: 45.7 x 45.7 mm, 33 parts, among them IC1 REG1117, IC2 REG1117, Q1 BUK98180-100A, Q2 BUK98180-100A, Q3 BUK98180-100A, Q4 BUK98180-100A, X1 53261-06

Commit message: Move the power connector further away from the SOC
Parts:
- moved CN1 2.50 mm to (10.7, 15.4)
Routing:
- net AC1: track 2.17 -> 4.37 mm
- net AC2: track 2.19 -> 4.36 mm
Changed lines of the file:
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@@
 <?xml version="1.0" encoding="utf-8"?>
 <!DOCTYPE eagle SYSTEM "eagle.dtd">
-<eagle version="7.5.0">
+<eagle version="7.4.0">
 <drawing>
 <settings>
@@
 <grid distance="0.00393700787" unitdist="inch" unit="inch" style="lines" multiple="1" display="no" altdistance="0.025" altunitdist="inch" altunit="inch"/>
 <layers>
-<layer number="1" name="Top" color="4" fill="1" visible="no" active="yes"/>
+<layer number="1" name="Top" color="4" fill="1" visible="yes" active="yes"/>
 <layer number="2" name="Route2" color="1" fill="3" visible="no" active="no"/>
 <layer number="3" name="Route3" color="4" fill="3" visible="no" active="no"/>
@@
 <attribute name="NAME" x="41.51" y="22.963" size="0.4064" layer="25"/>
 </element>
-<element name="CN1" library="adafruit" package="JST-PH-2-THM" value="" x="13.24" y="15.37" smashed="yes" rot="MR270"/>
+<element name="CN1" library="adafruit" package="JST-PH-2-THM" value="" x="10.74" y="15.37" smashed="yes" rot="MR270"/>
 <element name="IC1" library="burr-brown" package="SOT223" value="REG1117" x="31.83" y="17.75" smashed="yes" rot="R180">
 <attribute name="MPN" value="REG1117" x="31.83" y="17.75" size="1.778" layer="27" rot="R180" display="off"/>
@@
 <via x="5.6" y="19.3" extent="1-16" drill="0.6"/>
 <via x="9.8" y="19.3" extent="1-16" drill="0.6"/>
-<via x="10.7" y="15.9" extent="1-16" drill="0.6"/>
+<via x="12.1" y="12.6" extent="1-16" drill="0.6"/>
 <via x="9.7" y="22.3" extent="1-16" drill="0.6"/>
 <via x="6.7" y="23.3" extent="1-16" drill="0.6"/>
@@
 <contactref element="B2" pad="AC1"/>
 <contactref element="CN1" pad="1"/>
-<wire x1="13.24" y1="14.37" x2="13.24" y2="14.34" width="1.016" layer="1"/>
-<wire x1="13.24" y1="14.34" x2="14.75" y2="12.83" width="1.016" layer="1" curve="90"/>
+<wire x1="14.75" y1="12.83" x2="14" y2="12.8" width="1.016" layer="1"/>
+<wire x1="14" y1="12.8" x2="13.2" y2="13.2" width="1.016" layer="1" curve="-57.710717"/>
+<wire x1="13.2" y1="13.2" x2="10.74" y2="14.37" width="1.016" layer="1" curve="59.968301"/>
 </signal>
 <signal name="AC2">
 <contactref element="B2" pad="AC2"/>
 <contactref element="CN1" pad="2"/>
-<wire x1="13.24" y1="16.37" x2="13.24" y2="16.42" width="1.016" layer="1"/>
-<wire x1="13.24" y1="16.42" x2="14.75" y2="17.93" width="1.016" layer="1" curve="-90"/>
+<wire x1="14.75" y1="17.93" x2="14" y2="17.9" width="1.016" layer="1"/>
+<wire x1="14" y1="17.9" x2="12.8" y2="17.2" width="1.016" layer="1" curve="55.931116"/>
+<wire x1="12.8" y1="17.2" x2="10.74" y2="16.37" width="1.016" layer="1" curve="-72.553847"/>
 </signal>
 <signal name="GPIO12">
