File: LED-control.brd (EAGLE design)
At the start: 48.3 x 48.3 mm, 34 parts, among them IC1 REG1117, IC2 REG1117, U1 ATMEGA328P_TQFP

Commit message: Revise all the things
Parts:
- removed C12: 0.1uF, SparkFun-Passives:1206
- removed C6, C8: 10uF, SparkFun-Retired:EIA3216
- removed C7: 0.1uF, SparkFun-Capacitors:0603-CAP
- removed C9: .22uF, SparkFun-Retired:0402-CAP
- removed I2C: (no value), SparkFun-Connectors:JST-2-PTH-NS
- removed IC1, IC2: REG1117, burr-brown:SOT223
- removed LOGO1: OSHW-LOGOS, SparkFun-Aesthetics:OSHW-LOGO-S
- removed MPU: ESP8266_ESP-12, ESP8266-ESP12:ESP8266-ESP12
- removed R10, R11, R12, R13: 10k, SparkFun-Resistors:1206
- removed R6: (no value), SparkFun-Resistors:0603-RES
- removed U2: (no value), adafruit:TSSOP28
- removed Y2: (no value), SparkFun-FreqCtrl:CRYSTAL-SMD-5X3
- added B1: MB1S, rectifier:SOIC-4
- added C11: 10uF, SparkFun-Retired:EIA3216
- added C3: 0.1uf, rcl:C0805
- added FRAME1: (no value), SparkFun-Aesthetics:DUMMY
- added I2C1: (no value), SparkFun-Connectors:JST-2-PTH-NS
- added JP3: (no value), SparkFun-Connectors:1X06-SMD_EDGE
- added JP4: FEMALE 2x3, SparkFun-Connectors:2X3
- added LOGO2: OSHW-LOGOS, SparkFun-Aesthetics:OSHW-LOGO-S
- added PWR: red, SparkFun-LED:LED-0603
- added R7: 10k, rcl:R0805
- added REG3V, REG5V: REG1117, burr-brown:SOT223
- added U$1: ESP8266_ESP-12, ESP8266-ESP12:ESP8266-ESP12
- C1: value 10uF -> 0.1uf; device SparkFun-Capacitors:1206 -> rcl:C0805
- C10: value .22uF -> 0.1uF; device SparkFun-Retired:0402-CAP -> SparkFun-Capacitors:0603-CAP
- C2: value 10uF -> 0.1uF; device SparkFun-Capacitors:1206 -> SparkFun-Capacitors:0603-CAP
- C4: value 0.1uF -> 47uf; device SparkFun-Capacitors:0603-CAP -> SparkFun-Capacitors:PANASONIC_C
- C5: value 10uF -> 47uf; device SparkFun-Retired:EIA3216 -> SparkFun-Capacitors:PANASONIC_C
- JP1: device SparkFun-Connectors:JST-2-PTH-VERT -> SparkFun-Connectors:1X06_SMD_STRAIGHT_COMBO
- JP2: device SparkFun-Connectors:1X06-SIP_LOCK -> SparkFun-Connectors:JST-2-PTH-VERT
- R1: value 0 Ohm -> 330Ohm; device SparkFun-Resistors:0603-RES -> rcl:R0805
- R2, R4: value 0 Ohm -> 10k; device SparkFun-Resistors:0603-RES -> rcl:R0805
- R3: value 0 Ohm -> (none)
- R5: value (none) -> 10k; device SparkFun-Resistors:0603-RES -> rcl:R0805
- U1: value ATMEGA328P_TQFP -> (none); device SparkFun-DigitalIC:TQFP32-08 -> adafruit:TSSOP28
- moved C10 30.8 mm to (43.7, 18.3), turned to 315 degrees
- moved C4 28.5 mm to (32.5, 7.14), turned to 135 degrees
- moved C5 26.6 mm to (41.0, 15.2), turned to 135 degrees
- moved JP1 23.2 mm to (34.8, 22.5), turned to 315 degrees
- moved C1 22.3 mm to (33.0, 33.3), turned to 45 degrees
- moved JP2 20.0 mm to (27.1, 21.1), turned to 45 degrees
- moved R2 17.8 mm to (14.4, 23.3), turned to 225 degrees
- moved C2 12.9 mm to (29.8, 4.60), turned to 315 degrees
- moved R5 11.7 mm to (22.2, 36.8), turned to 45 degrees
- moved R4 10.2 mm to (19.4, 39.5), turned to 45 degrees
- moved R1 10.1 mm to (39.2, 33.5), turned to 225 degrees
- moved U1 7.30 mm to (22.1, 26.0), turned to 315 degrees
- moved R3 5.30 mm to (25.2, 29.4), turned to 315 degrees
Connections:
- removed net +3V3: C12.1, C6.A, C7.1, IC2.2, MPU.16, R10.1, R11.1, R12.1
- removed net AT_RXD: R1.1, R4.2, U1.30
- removed net AT_TXD: R2.1, R3.2, U1.31
- removed net ESP_RESET: MPU.9, R10.2
- removed net ESP_RXD: MPU.7, U1.32
- removed net ESP_SCL: MPU.5
- removed net ESP_SDA: MPU.6
- removed net ESP_TXD: MPU.8, U1.1
- removed net FTDI_RX: JP2.2, R2.2, R4.1
- removed net FTDI_TX: JP2.3, R1.2, R3.1
- removed net N$5: U1.19
- new net RX: JP1.2, JP3.2, JP4.5, U$1.7
- new net TX: JP1.3, JP3.3, JP4.6, U$1.8
- net #OE: now also R3.1, U1.23; no longer R6.1, U2.23
- net +5V: now also C4.+, JP4.4, REG3V.3, REG5V.2; no longer C1.1, C4.1, C5.A, IC1.2, IC2.3, JP2.4, R5.2, U1.18, U1.4, U1.6
- net 12V: now also B1.+, C11.A, JP1.6, JP3.6, JP4.1, REG5V.3; no longer C8.A, IC1.3, JP1.2
- net 3.3V: now also C1.1, C10.1, C3.1, C5.+, R1.2, R2.1, R3.2, R4.1, R5.1, REG3V.2, U$1.16, U1.28; no longer R6.2, U2.28
- net ADC: now also U$1.10; no longer MPU.10
- net BLUE: now also U1.7; no longer U2.7
- net CH_PD: now also R5.2, U$1.11; no longer MPU.11, R11.2
- net GND: now also B1.-, C10.2, C11.C, C3.2, C4.-, C5.-, JP3.1, JP4.3, PWR.C, R7.1, REG3V.1, REG5V.1, U$1.1, U1.1, U1.14, U1.2, U1.24, U1.25, U1.4; no longer C10.1, C12.2, C4.2, C5.C, C6.C, C7.2, C8.C, C9.1, IC1.1, IC2.1, JP2.6, MPU.1, R13.1, U1.21, U2.1, U2.14, U2.2, U2.24, U2.25, U2.3, U2.4, U2.5
- net GPIO0: now also JP1.5, JP3.5, JP4.2, R2.2, U$1.4; no longer MPU.4, R12.2
- net GPIO12: now also U$1.14; no longer MPU.14
- net GPIO13: now also U$1.15; no longer MPU.15
- net GPIO14: now also U$1.13; no longer MPU.13
- net GPIO15: now also R7.2, U$1.2; no longer MPU.2, R13.2
- net GPIO16: now also U$1.12; no longer MPU.12
- net GPIO2: now also U$1.3; no longer MPU.3
- net GREEN: now also U1.9; no longer U2.9
- net N$2: now also PWR.A, R1.1; no longer C9.2, U1.8, Y2.1
- net N$3: now also B1.~1, JP2.2; no longer C10.2, U1.7, Y2.3
- net N$4: now also B1.~2, JP2.1; no longer U1.22
- net RED: now also U1.8; no longer U2.8
- net RESET: now also JP1.4, JP3.4, R4.2, U$1.9; no longer JP2.1, R5.1, U1.29
- net SCL: now also I2C1.1, U$1.6, U1.26; no longer I2C.1, U1.28, U2.26
- net SDA: now also I2C1.2, U$1.5; no longer I2C.2, U2.27
- net WHITE: now also U1.15; no longer U2.15
Routing:
- net RX: track 0.00 -> 90.2 mm
- net TX: track 0.00 -> 83.2 mm
- net 3.3V: track 3.30 -> 76.0 mm, vias 0 -> 3
- net +3V3: track 62.0 -> 0.00 mm, vias 2 -> 0
- net +5V: track 82.8 -> 31.8 mm
- net GPIO0: track 6.06 -> 40.1 mm
- net AT_RXD: track 19.1 -> 0.00 mm
- net AT_TXD: track 16.0 -> 0.00 mm
- net WHITE: track 49.9 -> 34.5 mm
- net ESP_RXD: track 15.0 -> 0.00 mm, vias 1 -> 0
- net ESP_TXD: track 13.6 -> 0.00 mm, vias 1 -> 0
- net RESET: track 29.6 -> 41.5 mm, vias 0 -> 1
- net FTDI_TX: track 10.8 -> 0.00 mm, vias 1 -> 0
- net GREEN: track 12.3 -> 22.6 mm
- net ESP_RESET: track 8.90 -> 0.00 mm, vias 1 -> 0
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