File: LED-control.sch (EAGLE design)
At the start: 34 parts, among them IC1 REG1117, IC2 REG1117, U1 ATMEGA328P_TQFP

Commit message: Revise all the things
Parts:
- removed C12: 0.1uF, SparkFun-Passives:CAP1206
- removed C6, C8: 10uF, SparkFun-Retired:10UF-TANT
- removed C7: 0.1uF, SparkFun-Capacitors:0.1UF-25V(+80/-20%)(0603)
- removed C9: .22uF, SparkFun-Retired:.22UF-CER
- removed I2C: (no value), SparkFun-Connectors:M02-JST-2-PTH-NO_SILK
- removed IC1, IC2: REG1117, burr-brown:REG1117
- removed LOGO1: OSHW-LOGOS, SparkFun-Aesthetics:OSHW-LOGOS
- removed MPU: ESP8266_ESP-12, ESP8266-ESP12:ESP8266_ESP-12
- removed R10, R11, R12, R13: 10k, SparkFun-Resistors:RESISTOR1206
- removed R6: (no value), SparkFun-Resistors:RESISTOR0603
- removed U2: (no value), adafruit:PCA9685
- removed Y2: (no value), SparkFun-FreqCtrl:CRYSTAL5X3
- added B1: MB1S, rectifier:MB1S
- added C11: 10uF, SparkFun-Retired:10UF-TANT
- added C3: 0.1uf, rcl:C-EUC0805
- added FRAME1: (no value), SparkFun-Aesthetics:FRAME-LETTERNO_PACKAGE
- added I2C1: (no value), SparkFun-Connectors:M02-JST-2-PTH-NO_SILK
- added JP3: (no value), SparkFun-Connectors:M061X06-SMD_EDGE_FEMALE
- added JP4: FEMALE 2x3, SparkFun-Connectors:M03X2FEMALE
- added LOGO2: OSHW-LOGOS, SparkFun-Aesthetics:OSHW-LOGOS
- added PWR: red, SparkFun-LED:LED0603
- added R7: 10k, rcl:R-EU_R0805
- added REG3V, REG5V: REG1117, burr-brown:REG1117
- added U$1: ESP8266_ESP-12, ESP8266-ESP12:ESP8266_ESP-12
- C1: value 10uF -> 0.1uf; device SparkFun-Capacitors:10UF-6.3V-20%(1206) -> rcl:C-EUC0805
- C10: value .22uF -> 0.1uF; device SparkFun-Retired:.22UF-CER -> SparkFun-Capacitors:0.1UF-25V(+80/-20%)(0603)
- C2: value 10uF -> 0.1uF; device SparkFun-Capacitors:10UF-6.3V-20%(1206) -> SparkFun-Capacitors:0.1UF-25V(+80/-20%)(0603)
- C4: value 0.1uF -> 47uf; device SparkFun-Capacitors:0.1UF-25V(+80/-20%)(0603) -> SparkFun-Capacitors:CAP_POLC
- C5: value 10uF -> 47uf; device SparkFun-Retired:10UF-TANT -> SparkFun-Capacitors:CAP_POLC
- JP1: device SparkFun-Connectors:M02JST-PTH-VERT -> SparkFun-Connectors:M06SMD-STRAIGHT-COMBO-FEMALE
- JP2: device SparkFun-Connectors:M06SIP_LOCK -> SparkFun-Connectors:M02JST-PTH-VERT
- R1: value 0 Ohm -> 330Ohm; device SparkFun-Resistors:RESISTOR0603 -> rcl:R-EU_R0805
- R2, R4: value 0 Ohm -> 10k; device SparkFun-Resistors:RESISTOR0603 -> rcl:R-EU_R0805
- R3: value 0 Ohm -> (none)
- R5: value (none) -> 10k; device SparkFun-Resistors:RESISTOR0603 -> rcl:R-EU_R0805
- U1: value ATMEGA328P_TQFP -> (none); device SparkFun-DigitalIC:ATMEGA328P_TQFP -> adafruit:PCA9685
Connections:
- removed net +3V3: C12.1, C6.+, C7.1, IC2.VOUT, MPU.VCC, R10.1, R11.1, R12.1
- removed net AT_RXD: R1.1, R4.2, U1.PD0(RXD)
- removed net AT_TXD: R2.1, R3.2, U1.PD1(TXD)
- removed net ESP_RESET: MPU.REST, R10.2
- removed net ESP_RXD: MPU.RXD, U1.PD2(INT0)
- removed net ESP_SCL: MPU.GPIO5
- removed net ESP_SDA: MPU.GPIO4
- removed net ESP_TXD: MPU.TXD, U1.PD3(INT1)
- removed net FTDI_RX: JP2.2, R2.2, R4.1
- removed net FTDI_TX: JP2.3, R1.2, R3.1
- removed net N$5: U1.ADC6
- new net RX: JP1.2, JP3.2, JP4.5, U$1.RXD
- new net TX: JP1.3, JP3.3, JP4.6, U$1.TXD
- net #OE: now also R3.1, U1.#OE; no longer R6.1, U2.#OE
- net +5V: now also C4.+, JP4.4, REG3V.VIN, REG5V.VOUT; no longer C1.1, C4.1, C5.+, IC1.VOUT, IC2.VIN, JP2.4, R5.2, U1.AVCC, U1.VCC@4, U1.VCC@6
- net 12V: now also B1.+, C11.+, JP1.6, JP3.6, JP4.1, REG5V.VIN; no longer C8.+, IC1.VIN, JP1.2
- net 3.3V: now also C1.1, C10.1, C3.1, C5.+, R1.2, R2.1, R3.2, R4.1, R5.1, REG3V.VOUT, U$1.VCC, U1.VDD; no longer R6.2, U2.VDD
- net ADC: now also U$1.ADC; no longer MPU.ADC
- net BLUE: now also U1.PWM1; no longer U2.PWM1
- net CH_PD: now also R5.2, U$1.CH_PD; no longer MPU.CH_PD, R11.2
- net GND: now also B1.-, C10.2, C11.-, C3.2, C4.-, JP3.1, JP4.3, PWR.C, R7.1, REG3V.GND, REG5V.GND, U$1.GND, U1.A0, U1.A1, U1.A2, U1.A3, U1.A4, U1.A5, U1.EXTCLK, U1.GND; no longer C10.1, C12.2, C4.2, C6.-, C7.2, C8.-, C9.1, IC1.GND, IC2.GND, JP2.6, MPU.GND, R13.1, U1.AGND, U1.GND@3, U1.GND@5, U2.A0, U2.A1, U2.A2, U2.A3, U2.A4, U2.A5, U2.EXTCLK, U2.GND
- net GPIO0: now also JP1.5, JP3.5, JP4.2, R2.2, U$1.GPIO0; no longer MPU.GPIO0, R12.2
- net GPIO12: now also U$1.GPIO12; no longer MPU.GPIO12
- net GPIO13: now also U$1.GPIO13; no longer MPU.GPIO13
- net GPIO14: now also U$1.GPIO14; no longer MPU.GPIO14
- net GPIO15: now also R7.2, U$1.GPIO15; no longer MPU.GPIO15, R13.2
- net GPIO16: now also U$1.GPIO16; no longer MPU.GPIO16
- net GPIO2: now also U$1.GPIO2; no longer MPU.GPIO2
- net GREEN: now also U1.PWM3; no longer U2.PWM3
- net N$2: now also PWR.A, R1.1; no longer C9.2, U1.PB7(XTAL2/TOSC2), Y2.1
- net N$3: now also B1.AC1, JP2.2; no longer C10.2, U1.PB6(XTAL1/TOSC1), Y2.2
- net N$4: now also B1.AC2, JP2.1; no longer U1.ADC7
- net RED: now also U1.PWM2; no longer U2.PWM2
- net RESET: now also JP1.4, JP3.4, R4.2, U$1.REST; no longer JP2.1, R5.1, U1.PC6(/RESET)
- net SCL: now also I2C1.1, U$1.GPIO4, U1.SCL; no longer I2C.1, U1.PC5(ADC5/SCL), U2.SCL
- net SDA: now also I2C1.2, U$1.GPIO5, U1.SDA; no longer I2C.2, U1.PC4(ADC4/SDA), U2.SDA
- net WHITE: now also U1.PWM8; no longer U2.PWM8
Other:
- note added: "Processor"
- note added: "Pullups"
