File: Programmer.sch (EAGLE design)
At the start: 31 parts

Commit message: mk9 brah.
Parts:
- removed B1: MB1S, rectifier:MB1S
- removed I2C1: (no value), SparkFun-Connectors:M02-JST-2-PTH-NO_SILK
- removed JP2: (no value), SparkFun-Connectors:M02JST-PTH-VERT
- removed JP3: (no value), SparkFun-Connectors:M061X06-SMD_EDGE_FEMALE
- removed PWR: red, SparkFun-LED:LED0603
- removed R2, R4, R5, R7: 10k, rcl:R-EU_R0805
- removed R3: (no value), SparkFun-Resistors:RESISTOR0603
- removed SV1, SV2: (no value), con-lstb:MA04-1
- removed U1: (no value), adafruit:PCA9685
- added 12VDC: (no value), SparkFun-Connectors:M023.5MM
- added ALWAYS_PROGRAMMING, CONNECT_5V_TOGETHER: (no value), SparkFun-Connectors:M02LOCK
- added C6: 22pf, SparkFun-Capacitors:CAP1206
- added H3, H4, H5, H6: MOUNT-HOLE3.0, holes:MOUNT-HOLE3.0
- added PRG, RESET: SWITCH-MOMENTARY-2PTH, SparkFun-Electromechanical:SWITCH-MOMENTARY-2PTH
- added TX_RX_FLIBBLER: (no value), SparkFun-Connectors:M03X2NO_SILK
- added U$2: CH340G, CH340G-USB-SERIAL:CH340G
- added USB: USB-SMD-NS, SparkFun-Connectors:USB-SMD-NS
- added Y1: 12mhz, SparkFun-FreqCtrl:CRYSTALSMD
- C1: value 0.1uf -> 22pf; device rcl:C-EUC0805 -> SparkFun-Capacitors:CAP1206
- C3: value 0.1uf -> 0.1uF; device rcl:C-EUC0805 -> rcl:C-EUC1206K
- JP1: value (none) -> RASPBERRYPI-B+-GPIO; device SparkFun-Connectors:M06SMD-STRAIGHT-COMBO-FEMALE -> SparkFun-Boards:RASPBERRYPI-B+-GPIO
- R1: value 330Ohm -> (none); device rcl:R-EU_R0805 -> rcl:R-EU_0207/12
- U$1: value ESP8266_ESP-12 -> RELAYPTH4; device ESP8266-ESP12:ESP8266_ESP-12 -> SparkFun-Electromechanical:RELAYPTH4
- renumbered JP5 to I2C
Connections:
- removed net #OE: R3.1, U1.#OE
- removed net ADC: U$1.ADC
- removed net BLUE: SV1.3, U1.PWM1
- removed net CH_PD: R5.2, U$1.CH_PD
- removed net GPIO12: U$1.GPIO12
- removed net GPIO13: U$1.GPIO13
- removed net GPIO14: U$1.GPIO14
- removed net GPIO15: R7.2, U$1.GPIO15
- removed net GPIO16: U$1.GPIO16
- removed net GPIO2: U$1.GPIO2
- removed net GREEN: SV1.1, U1.PWM3
- removed net N$2: PWR.A, R1.1
- removed net N$3: B1.AC1, JP2.2
- removed net RED: SV1.2, U1.PWM2
- removed net RESET: JP1.4, JP3.4, R4.2, U$1.REST
- removed net WHITE: SV2.4, U1.PWM8
- new net +5V_REMOTE: CONNECT_5V_TOGETHER.2, JP4.4
- new net 12V_REMOTE: JP4.1, U$1.MAIN
- new net NC1: JP1.5V@2
- new net NC2: JP1.5V@4
- new net NC3: JP1.3.3V@1
- new net NC4: JP1.3.3V@17
- new net OSCI: C1.1, U$2.XI, Y1.1
- new net OSCO: C6.1, U$2.XO, Y1.2
- new net RESET_RELAY: RESET.2, U$1.COIL1
- new net RPI_RX: JP1.RXI, TX_RX_FLIBBLER.3
- new net RPI_TX: JP1.TXO, TX_RX_FLIBBLER.4
- new net USB_D+: U$2.D+, USB.D+
- new net USB_D-: U$2.D-, USB.D-
- net +5V: now also CONNECT_5V_TOGETHER.1, RESET.1; no longer JP4.4
- net 12V: now also 12VDC.2, U$1.NC; no longer B1.+, JP1.6, JP3.6, JP4.1, SV1.4
- net 3.3V: now also U$2.V3, U$2.VCC; no longer C1.1, R1.2, R2.1, R3.2, R4.1, R5.1, U$1.VCC, U1.VDD
- net GND: now also 12VDC.1, ALWAYS_PROGRAMMING.2, C6.2, JP1.GND@14, JP1.GND@20, JP1.GND@25, JP1.GND@30, JP1.GND@34, JP1.GND@39, JP1.GND@6, JP1.GND@9, PRG.1, R1.1, U$1.COIL2, U$2.GND, USB.GND; no longer B1.-, JP1.1, JP3.1, PWR.C, R7.1, SV2.1, SV2.2, SV2.3, U$1.GND, U1.A0, U1.A1, U1.A2, U1.A3, U1.A4, U1.A5, U1.EXTCLK, U1.GND
- net GPIO0: now also ALWAYS_PROGRAMMING.1, PRG.2; no longer JP1.5, JP3.5, R2.2, U$1.GPIO0
- net N$4: now also R1.2, U$1.NO; no longer B1.AC2, JP2.1
- net RX: now also TX_RX_FLIBBLER.2, TX_RX_FLIBBLER.5, U$2.TX; no longer JP1.2, JP3.2, U$1.RXD
- net SCL: now also JP1.SCL; no longer I2C1.1, U$1.GPIO4, U1.SCL
- net SDA: now also JP1.SDA; no longer I2C1.2, U$1.GPIO5, U1.SDA
- net TX: now also TX_RX_FLIBBLER.1, TX_RX_FLIBBLER.6, U$2.RX; no longer JP1.3, JP3.3, U$1.TXD
Other:
- note removed: "Diagnostic LEDs + Programming Port"
- note removed: "Processor"
- note removed: "Pullups"
- moved on the sheet: C1, C3, R1

Commit message: mk10
Parts:
- removed ALWAYS_PROGRAMMING, CONNECT_5V_TOGETHER: (no value), SparkFun-Connectors:M02LOCK
- removed H3, H4, H5, H6: MOUNT-HOLE3.0, holes:MOUNT-HOLE3.0
- removed I2C: (no value), SparkFun-Connectors:M03PTH
- removed JP1: RASPBERRYPI-B+-GPIO, SparkFun-Boards:RASPBERRYPI-B+-GPIO
- removed JP4: FEMALE 2x3, SparkFun-Connectors:M03X2FEMALE
- removed R1: (no value), rcl:R-EU_0207/12
- removed TX_RX_FLIBBLER: (no value), SparkFun-Connectors:M03X2NO_SILK
- removed U$1: RELAYPTH4, SparkFun-Electromechanical:RELAYPTH4
- added C7: 10uF, SparkFun-Retired:10UF-TANT
- added C8: 0.1uF, SparkFun-Capacitors:0.1UF-25V(+80/-20%)(0603)
- added C9: 47uf, SparkFun-Capacitors:CAP_POLC
- added J1: (no value), SparkFun-Connectors:CONN_03X22X3_SILK_MALE_PTH
- added J2: (no value), SparkFun-Connectors:CONN_05X2SHD
- added J3, J4: (no value), SparkFun-Connectors:CONN_03LOCK
- added PCB1: RPI3, e14_Rpi3_RevA:RPI3
- added REG5V1: REG1117, burr-brown:REG1117
Connections:
- removed net +5V_REMOTE: CONNECT_5V_TOGETHER.2, JP4.4
- removed net 12V_REMOTE: JP4.1, U$1.MAIN
- removed net N$4: R1.2, U$1.NO
- removed net NC1: JP1.5V@2
- removed net NC2: JP1.5V@4
- removed net NC3: JP1.3.3V@1
- removed net NC4: JP1.3.3V@17
- removed net RESET_RELAY: RESET.2, U$1.COIL1
- removed net RPI_RX: JP1.RXI, TX_RX_FLIBBLER.3
- removed net RPI_TX: JP1.TXO, TX_RX_FLIBBLER.4
- new net C_RX: J1.5, U$2.TX
- new net C_TX: J1.6, U$2.RX
- new net L_RX: J2.4, J4.2
- new net L_TX: J2.2, J3.2
- new net RESET: J2.10, RESET.2
- new net RPI_5V: C8.1, C9.+, PCB1.5V@2, PCB1.5V@4, REG5V1.VOUT
- new net R_RX: J1.1, PCB1.GPIO14
- new net R_TX: J1.2, PCB1.GPIO15
- net +5V: now also J2.7; no longer CONNECT_5V_TOGETHER.1, RESET.1
- net 12V: now also C7.+, J2.9, REG5V1.VIN; no longer U$1.NC
- net 3.3V: now also J2.5
- net GND: now also C7.-, C8.2, C9.-, J2.6, PCB1.GND@14, PCB1.GND@20, PCB1.GND@25, PCB1.GND@30, PCB1.GND@34, PCB1.GND@39, PCB1.GND@6, PCB1.GND@9, REG5V1.GND, RESET.1; no longer ALWAYS_PROGRAMMING.2, I2C.2, JP1.GND@14, JP1.GND@20, JP1.GND@25, JP1.GND@30, JP1.GND@34, JP1.GND@39, JP1.GND@6, JP1.GND@9, JP4.3, R1.1, U$1.COIL2
- net GPIO0: now also J2.8; no longer ALWAYS_PROGRAMMING.1, JP4.2
- net RX: now also J1.3, J3.1, J4.3; no longer JP4.5, TX_RX_FLIBBLER.2, TX_RX_FLIBBLER.5, U$2.TX
- net SCL: now also J2.1; no longer I2C.3, JP1.SCL
- net SDA: now also J2.3; no longer I2C.1, JP1.SDA
- net TX: now also J1.4, J3.3, J4.1; no longer JP4.6, TX_RX_FLIBBLER.1, TX_RX_FLIBBLER.6, U$2.RX
